File: backlight_controller_6x3.kicad_pcb (KiCad board)
At the start: 2 copper layers, 121.3 x 67.3 mm, 84 parts, among them J1 HEADER_01X25_MALE, J10 M12-5-RCPT, J11 M12-5-RCPT, J12 M12-5-RCPT, J2 HEADER_01X25_MALE, J3 DB9F, J4 DB9M, J5 M12-5-RCPT, J6 M12-5-RCPT, J7 M12-5-RCPT, J8 M12-5-RCPT, J9 M12-5-RCPT, P1 MINI_FIT, U1 SN74ABT541BDWR, U10 NUD3124, U2 SN74ABT541BDWR, U3 NUD3124, U4 NUD3124, U5 NUD3124, U6 NUD3124, U7 NUD3124, U8 NUD3124, U9 NUD3124

Commit message: Update version documentation
Routing:
- net GND: track 757.9 -> 0.00 mm, vias 4 -> 0
- net VAA: track 338.4 -> 0.00 mm, vias 1 -> 0
- net VEE: track 125.6 -> 0.00 mm, vias 3 -> 0
- net /CHANNEL_9: track 95.2 -> 0.00 mm
- net /CHANNEL_11: track 92.2 -> 0.00 mm
- net /~ENABLE: track 90.0 -> 0.00 mm, vias 2 -> 0
- net /CHANNEL_10: track 86.7 -> 0.00 mm
- net /CHANNEL_0: track 84.0 -> 0.00 mm
- net VDD: track 82.0 -> 0.00 mm
- net /backlight_6x3/C_13: track 79.1 -> 0.00 mm, vias 1 -> 0
- net /backlight_6x3/C_0: track 78.5 -> 0.00 mm, vias 1 -> 0
- net /CHANNEL_8: track 76.8 -> 0.00 mm, vias 1 -> 0
- net /CHANNEL_1: track 76.8 -> 0.00 mm
- net /backlight_6x3/C_1: track 74.8 -> 0.00 mm, vias 3 -> 0
- net /backlight_6x3/C_8: track 71.5 -> 0.00 mm, vias 3 -> 0
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- removed copper zone on B.Cu, net GND
- removed copper zone on F.Cu, net VAA
Other:
- board text added: "Janelia Modular Device backlight_controller part_number: 1272 06/2019 ver 1.0 6x3"
- board text removed: "Janelia Modular Device backlight_controller part_number: 1270 05/2019 ver 1.3 6x3"

Commit message: Prerouting
Parts:
- removed D18: LED_GRN, backlight_controller_6x3:LED0805
- removed J11, J12: M12-5-RCPT, backlight_controller_6x3:M12-5_RCPT_F_SMD
- added C7: 0.1uF, backlight_controller_6x3:SM0805, B.Cu at (83.8, 94.6)
- added C8: 0.1uF, backlight_controller_6x3:SM0805, B.Cu at (83.8, 84.5)
- added C9: 0.1uF, backlight_controller_6x3:SM0805, B.Cu at (73.7, 88.9)
- added R26: 287, backlight_controller_6x3:SM0805, B.Cu at (178.4, 132.7)
- added REG1: CONV_DC_DC_5V_1A, backlight_controller_6x3:DC_DC_CONV_R78C, F.Cu at (109.9, 78.7)
- added SW1: VAL**, backlight_controller_6x3:SWITCH_KT, F.Cu at (83.8, 78.1)
- added SW2: VAL**, backlight_controller_6x3:SWITCH_KT, F.Cu at (96.5, 78.1)
- added TEENSY1: TEENSY_3.5, backlight_controller_6x3:TEENSY_3.5_MIN, F.Cu at (61.0, 92.7)
- added U11: NUD3124, backlight_controller_6x3:TO-236-3, B.Cu at (178.4, 128.9)
- added U12: VAL**, backlight_controller_6x3:MAX6817, B.Cu at (73.7, 85.7)
- C1, C2: value 0.1uF -> 10uF
- D1: value DIODE_10A -> LED_GRN; footprint backlight_controller_6x3:CFP15 -> backlight_controller_6x3:LED0805; moved to F.Cu
- J1: value HEADER_01X25_MALE -> DB9F; footprint backlight_controller_6x3:HEADER_01x25 -> backlight_controller_6x3:DB9F_SMD; moved to F.Cu
- J2: value HEADER_01X25_MALE -> DB9M; footprint backlight_controller_6x3:HEADER_01x25 -> backlight_controller_6x3:DB9M_SMD; moved to F.Cu
- J3: value DB9F -> M12-5-RCPT; footprint backlight_controller_6x3:DB9F_SMD -> backlight_controller_6x3:M12-5_RCPT_F_SMD
- J4: value DB9M -> M12-5-RCPT; footprint backlight_controller_6x3:DB9M_SMD -> backlight_controller_6x3:M12-5_RCPT_F_SMD
- R1, R19, R20, R21, R22, R23, R24, R25: moved to B.Cu
- R10, R2, R4, R6, R8: value 287 -> 5.9k; moved to B.Cu
- R11, R13, R15, R17: value 75 -> 287
- R12, R14, R16, R18: value 287 -> 75; moved to B.Cu
- R3, R5, R7, R9: value 5.9k -> 287
- moved D1 119.6 mm to (189.2, 119.4)
- moved D2 110.0 mm to (79.4, 128.3), turned to 0 degrees
- moved U2 96.1 mm to (61.0, 92.7)
- moved U1 70.7 mm to (61.0, 118.1), turned to 0 degrees
- moved U3 63.0 mm to (58.4, 77.5), turned to 90 degrees
- moved D12 57.8 mm to (140.3, 78.1), turned to 90 degrees
- moved D16 57.8 mm to (178.4, 78.1), turned to 90 degrees
- moved D14 57.8 mm to (159.4, 78.1), turned to 90 degrees
- moved R20 56.5 mm to (121.3, 132.7), turned to 270 degrees
- moved R22 56.5 mm to (140.3, 132.7), turned to 270 degrees
- moved R24 56.5 mm to (159.4, 132.7), turned to 270 degrees
- moved R19 54.8 mm to (121.3, 78.1), turned to 270 degrees
- moved R21 54.8 mm to (140.3, 78.1), turned to 270 degrees
- moved R23 54.8 mm to (159.4, 78.1), turned to 270 degrees
- moved R25 54.8 mm to (178.4, 78.1), turned to 270 degrees
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Connections:
- C1 pad 1: VEE -> VAA
- C3 pad 1: VDD -> VEE
- C4 pad 1: VDD -> VEE
- C5 pad 1: VDD -> VAA
- C6 pad 1: VDD -> VAA
- D1 pad 1: VDD -> Net-(D1-Pad1)
- D1 pad 2: VAA -> GND
- HPS1 pad 1: VDD -> VAA
- HPS1 pad 4: Net-(HPS1-Pad4) -> (no net)
- HPS2 pad 1: VDD -> VAA
- HPS2 pad 4: Net-(HPS2-Pad4) -> (no net)
- HPS3 pad 1: VDD -> VAA
- HPS3 pad 4: Net-(HPS3-Pad4) -> (no net)
- HPS4 pad 1: VDD -> VAA
- HPS4 pad 4: Net-(HPS4-Pad4) -> (no net)
- J1 pad 1: VDD -> VAA
- J1 pad 2: GND -> /backlight_6x3/high_voltage_outputs/OUTPUT_0
- J1 pad 3: /A10 -> VAA
- J1 pad 4: /A11 -> /backlight_6x3/high_voltage_outputs/OUTPUT_1
- J1 pad 5: /CHANNEL_0 -> VAA
- J1 pad 6: /D55 -> /backlight_6x3/high_voltage_outputs/OUTPUT_2
- J1 pad 7: /D54.CS2 -> VAA
- J1 pad 8: /CHANNEL_1 -> /backlight_6x3/high_voltage_outputs/OUTPUT_3
- J1 pad 9: /CHANNEL_2 -> VAA
- J10 pad 2: /backlight_6x3/backlight_outputs/visible_2/NPN -> /backlight_6x3/backlight_outputs/visible_3/NPN
- J10 pad 4: Net-(J10-Pad4) -> (no net)
- J2 pad 1: /AREF -> GND
- J2 pad 2: VEE -> /backlight_6x3/low_voltage_outputs/OUTPUT_0
- J2 pad 3: /AGND -> GND
- J2 pad 4: /3.3V_250mA -> /backlight_6x3/low_voltage_outputs/OUTPUT_1
- J2 pad 5: /CHANNEL_11 -> GND
- J2 pad 6: /CHANNEL_10 -> /backlight_6x3/low_voltage_outputs/OUTPUT_2
- J2 pad 7: /CHANNEL_9 -> GND
- J2 pad 8: /CHANNEL_8 -> /backlight_6x3/low_voltage_outputs/OUTPUT_3
- J2 pad 9: /CHANNEL_7 -> GND
- J3 pad 2: /backlight_6x3/high_voltage_outputs/OUTPUT_0 -> /backlight_6x3/backlight_outputs/ir_0/NPN
- J3 pad 3: VAA -> GND
- J3 pad 4: /backlight_6x3/high_voltage_outputs/OUTPUT_1 -> (no net)
- J4 pad 1: GND -> VAA
- J4 pad 2: /backlight_6x3/low_voltage_outputs/OUTPUT_0 -> /backlight_6x3/backlight_outputs/visible_0/NPN
- J4 pad 4: /backlight_6x3/low_voltage_outputs/OUTPUT_1 -> (no net)
- J4 pad 5: GND -> VAA
- J5 pad 2: /backlight_6x3/backlight_outputs/ir_0/NPN -> /backlight_6x3/backlight_outputs/ir_1/NPN
- J5 pad 4: Net-(J5-Pad4) -> (no net)
- J6 pad 2: /backlight_6x3/backlight_outputs/visible_0/NPN -> /backlight_6x3/backlight_outputs/visible_1/NPN
- J6 pad 4: Net-(J6-Pad4) -> (no net)
- J7 pad 2: /backlight_6x3/backlight_outputs/ir_1/NPN -> /backlight_6x3/backlight_outputs/ir_2/NPN
- J7 pad 4: Net-(J7-Pad4) -> (no net)
- J8 pad 2: /backlight_6x3/backlight_outputs/visible_1/NPN -> /backlight_6x3/backlight_outputs/visible_2/NPN
- J8 pad 4: Net-(J8-Pad4) -> (no net)
- J9 pad 2: /backlight_6x3/backlight_outputs/ir_2/NPN -> /backlight_6x3/backlight_outputs/ir_3/NPN
- J9 pad 4: Net-(J9-Pad4) -> (no net)
- MH1 pad 1: Net-(MH1-Pad1) -> (no net)
- MH2 pad 1: Net-(MH2-Pad1) -> (no net)
- MH3 pad 1: Net-(MH3-Pad1) -> (no net)
- MH4 pad 1: Net-(MH4-Pad1) -> (no net)
- R1 pad 2: Net-(D2-Pad1) -> Net-(D1-Pad1)
- R10 pad 1: /backlight_6x3/C_4 -> /backlight_6x3/C_3
- R10 pad 2: Net-(D7-Pad1) -> /backlight_6x3/high_voltage_outputs/high_voltage_output_3/FAULT
- R11 pad 2: /backlight_6x3/low_voltage_outputs/OUTPUT_0 -> Net-(D6-Pad1)
- R12 pad 1: /backlight_6x3/C_5 -> /backlight_6x3/C_4
- R12 pad 2: Net-(D8-Pad1) -> /backlight_6x3/low_voltage_outputs/OUTPUT_0
- R13 pad 2: /backlight_6x3/low_voltage_outputs/OUTPUT_1 -> Net-(D7-Pad1)
- R14 pad 1: /backlight_6x3/C_6 -> /backlight_6x3/C_5
- R14 pad 2: Net-(D9-Pad1) -> /backlight_6x3/low_voltage_outputs/OUTPUT_1
- R15 pad 2: /backlight_6x3/low_voltage_outputs/OUTPUT_2 -> Net-(D8-Pad1)
- R16 pad 1: /backlight_6x3/C_7 -> /backlight_6x3/C_6
- R16 pad 2: Net-(D10-Pad1) -> /backlight_6x3/low_voltage_outputs/OUTPUT_2
- R17 pad 2: /backlight_6x3/low_voltage_outputs/OUTPUT_3 -> Net-(D9-Pad1)
- R18 pad 1: /backlight_6x3/C_8 -> /backlight_6x3/C_7
- R18 pad 2: Net-(D11-Pad1) -> /backlight_6x3/low_voltage_outputs/OUTPUT_3
- R19 pad 1: /backlight_6x3/C_9 -> /backlight_6x3/C_8
- R19 pad 2: Net-(D12-Pad1) -> Net-(D10-Pad1)
- R2 pad 1: /backlight_6x3/C_0 -> VEE
- R2 pad 2: Net-(D3-Pad1) -> /backlight_6x3/~ENABLE
- R20 pad 1: /backlight_6x3/C_10 -> /backlight_6x3/C_9
- R20 pad 2: Net-(D13-Pad1) -> Net-(D11-Pad1)
- R21 pad 1: /backlight_6x3/C_11 -> /backlight_6x3/C_10
- R21 pad 2: Net-(D14-Pad1) -> Net-(D12-Pad1)
- R22 pad 1: /backlight_6x3/C_12 -> /backlight_6x3/C_11
- R22 pad 2: Net-(D15-Pad1) -> Net-(D13-Pad1)
- R23 pad 1: /backlight_6x3/C_13 -> /backlight_6x3/C_12
- R23 pad 2: Net-(D16-Pad1) -> Net-(D14-Pad1)
- R24 pad 1: /backlight_6x3/C_14 -> /backlight_6x3/C_13
- R24 pad 2: Net-(D17-Pad1) -> Net-(D15-Pad1)
- R25 pad 1: /backlight_6x3/C_15 -> /backlight_6x3/C_14
- R25 pad 2: Net-(D18-Pad1) -> Net-(D16-Pad1)
- R3 pad 2: /backlight_6x3/high_voltage_outputs/high_voltage_output_0/FAULT -> Net-(D2-Pad1)
- R4 pad 1: /backlight_6x3/C_1 -> /backlight_6x3/C_0
- R4 pad 2: Net-(D4-Pad1) -> /backlight_6x3/high_voltage_outputs/high_voltage_output_0/FAULT
- R5 pad 2: /backlight_6x3/high_voltage_outputs/high_voltage_output_1/FAULT -> Net-(D3-Pad1)
- R6 pad 1: /backlight_6x3/C_2 -> /backlight_6x3/C_1
- R6 pad 2: Net-(D5-Pad1) -> /backlight_6x3/high_voltage_outputs/high_voltage_output_1/FAULT
- R7 pad 2: /backlight_6x3/high_voltage_outputs/high_voltage_output_2/FAULT -> Net-(D4-Pad1)
- R8 pad 1: /backlight_6x3/C_3 -> /backlight_6x3/C_2
- R8 pad 2: Net-(D6-Pad1) -> /backlight_6x3/high_voltage_outputs/high_voltage_output_2/FAULT
- R9 pad 2: /backlight_6x3/high_voltage_outputs/high_voltage_output_3/FAULT -> Net-(D5-Pad1)
- U1 pad 1: /~ENABLE -> /backlight_6x3/~ENABLE
- U10 pad 1: /backlight_6x3/C_15 -> /backlight_6x3/C_14
- U10 pad 3: /backlight_6x3/backlight_outputs/visible_3/NPN -> /backlight_6x3/backlight_outputs/ir_3/NPN
- U2 pad 1: /~ENABLE -> /backlight_6x3/~ENABLE
- U3 pad 1: /backlight_6x3/C_8 -> /ENABLE
- U3 pad 3: /backlight_6x3/backlight_outputs/ir_0/NPN -> /backlight_6x3/~ENABLE
- U4 pad 1: /backlight_6x3/C_9 -> /backlight_6x3/C_8
- U4 pad 3: /backlight_6x3/backlight_outputs/visible_0/NPN -> /backlight_6x3/backlight_outputs/ir_0/NPN
- U5 pad 1: /backlight_6x3/C_10 -> /backlight_6x3/C_9
- U5 pad 3: /backlight_6x3/backlight_outputs/ir_1/NPN -> /backlight_6x3/backlight_outputs/visible_0/NPN
- U6 pad 1: /backlight_6x3/C_11 -> /backlight_6x3/C_10
- U6 pad 3: /backlight_6x3/backlight_outputs/visible_1/NPN -> /backlight_6x3/backlight_outputs/ir_1/NPN
- U7 pad 1: /backlight_6x3/C_12 -> /backlight_6x3/C_11
- U7 pad 3: /backlight_6x3/backlight_outputs/ir_2/NPN -> /backlight_6x3/backlight_outputs/visible_1/NPN
- U8 pad 1: /backlight_6x3/C_13 -> /backlight_6x3/C_12
- U8 pad 3: /backlight_6x3/backlight_outputs/visible_2/NPN -> /backlight_6x3/backlight_outputs/ir_2/NPN
- U9 pad 1: /backlight_6x3/C_14 -> /backlight_6x3/C_13
- U9 pad 3: /backlight_6x3/backlight_outputs/ir_3/NPN -> /backlight_6x3/backlight_outputs/visible_2/NPN
Other:
- board size 121.3 x 67.3 mm -> 139.7 x 67.3 mm
- board text removed: "VDD"
- board text removed: "VEE"

Commit message: Route board
Parts:
- moved D1 23.5 mm to (189.2, 95.9)
- moved R1 23.5 mm to (189.2, 95.9)
Routing:
- net GND: track 0.00 -> 889.1 mm, vias 0 -> 2
- net VAA: track 0.00 -> 468.7 mm, vias 0 -> 5
- net /backlight_6x3/C_14: track 0.00 -> 160.0 mm
- net /backlight_6x3/C_15: track 0.00 -> 155.4 mm, vias 0 -> 2
- net /backlight_6x3/C_11: track 0.00 -> 140.4 mm
- net /backlight_6x3/C_13: track 0.00 -> 134.9 mm, vias 0 -> 2
- net /backlight_6x3/C_12: track 0.00 -> 127.5 mm, vias 0 -> 2
- net VEE: track 0.00 -> 110.1 mm, vias 0 -> 4
- net /backlight_6x3/C_3: track 0.00 -> 94.1 mm
- net /backlight_6x3/C_10: track 0.00 -> 81.8 mm, vias 0 -> 2
- net /backlight_6x3/C_9: track 0.00 -> 77.5 mm, vias 0 -> 2
- net /backlight_6x3/C_6: track 0.00 -> 72.5 mm, vias 0 -> 2
- net /backlight_6x3/C_7: track 0.00 -> 69.4 mm, vias 0 -> 2
- net /backlight_6x3/C_5: track 0.00 -> 67.5 mm, vias 0 -> 2
- net /backlight_6x3/C_8: track 0.00 -> 66.8 mm, vias 0 -> 2
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Other:
- net class LEDPOWER: clearance 0.254 -> 0.2032
- net class POWER: clearance 0.254 -> 0.2032
- net class SUPERPOWER: clearance 0.254 -> 0.2032

Commit message: Route board and generate gerbers
Parts:
- moved FID1 0.63 mm to (52.1, 73.0)
- moved FID4 0.63 mm to (52.1, 137.8)
Routing:
- net GND: track 889.1 -> 891.0 mm
- net VAA: track 468.7 -> 469.9 mm
- added copper zone on B.Cu, net GND
- added copper zone on F.Cu, net VAA
Other:
- board size 139.7 x 67.3 mm -> 140.3 x 67.3 mm
- board text added: "Both USB power and 24V power must be connected for board to operate!"
